Commit message: fix mesh paths

File: src/r6bot_description/urdf/r6bot.urdf (robot description, URDF)
Before this commit: robot r6bot, 8 links, 7 joints
Links:
- link link_1: geometry collision mesh filename=package://r6bot_description/meshes/link_1_collision.stl; visual mesh filename=package://r6bot_description/meshes/link_1_visual.stl
- link link_2: geometry collision mesh filename=package://r6bot_description/meshes/link_2_collision.stl; visual mesh filename=package://r6bot_description/meshes/link_2_visual.stl
- link link_3: geometry collision mesh filename=package://r6bot_description/meshes/link_3_collision.stl; visual mesh filename=package://r6bot_description/meshes/link_3_visual.stl
- link link_4: geometry collision mesh filename=package://r6bot_description/meshes/link_4_collision.stl; visual mesh filename=package://r6bot_description/meshes/link_4_visual.stl
- link link_5: geometry collision mesh filename=package://r6bot_description/meshes/link_5_collision.stl; visual mesh filename=package://r6bot_description/meshes/link_5_visual.stl
- link link_6: geometry collision mesh filename=package://r6bot_description/meshes/link_6_collision.stl; visual mesh filename=package://r6bot_description/meshes/link_6_visual.stl
- link link_7: geometry collision mesh filename=package://r6bot_description/meshes/link_7_collision.stl; visual mesh filename=package://r6bot_description/meshes/link_7_visual.stl
