Commit message: fix build script

File: src/r6bot_description/urdf/robot.urdf (robot description, URDF)
Before this commit: robot r6bot, 8 links, 7 joints
Links:
- added link tool0_tcp, mass 1e-9
- added link tool1_tcp, mass 1e-9
- link link_1: mass 0.461414 -> 0.552681
- link link_2: mass 0.331666 -> 0.423847
- link link_3: mass 0.498148 -> 0.573947
- link link_4: mass 0.216205 -> 0.28613
- link link_5: mass 0.363068 -> 0.367859
- link link_6: mass 0.15061 -> 0.164337
- link link_7: mass 0.171084 -> 0.117107
Joints:
- added joint tool0_tcp_frame: type fixed, parent link_7, child tool0_tcp, origin xyz=-6.41848e-17 8.44637e-18 0.047085 rpy=-9.35725e-16 -1.99408e-15 -1.96146e-29, axis 0 0 0
- added joint tool1_tcp_frame: type fixed, parent link_7, child tool1_tcp, origin xyz=-2.15106e-16 2.25417e-16 0.106885 rpy=-2.58091e-15 6.24476e-15 1.5708, axis 0 0 0
- joint joint_1: limit lower=0 upper=6.28319 effort=10 velocity=10 -> lower=-3.14159 upper=3.14159 effort=10 velocity=10; origin xyz=-6.00804e-17 5.03629e-17 0.1245 rpy=3.14159 -2.21112e-32 3.14159 -> xyz=7.33525e-17 9.71219e-17 0.1245 rpy=3.14159 -0 1.5708
- joint joint_2: limit lower=-3.91499 upper=2.3682 effort=10 velocity=10 -> lower=-3.14159 upper=3.14159 effort=10 velocity=10; origin xyz=1.83707e-15 -0.0895 -0.0575 rpy=-1.5708 2.22045e-16 1.94096e-14 -> xyz=1.2576e-16 0.0895 -0.0575 rpy=1.5708 1.3735e-16 -2.25307e-15
- joint joint_3: limit lower=-4.74747 upper=1.53571 effort=10 velocity=10 -> lower=-3.14159 upper=3.14159 effort=10 velocity=10; origin xyz=-0.139714 0.143108 0.0259997 rpy=-3.14159 2.36039e-15 -0.832485 -> xyz=4.2689e-08 -0.2 0.0259997 rpy=3.14159 4.65589e-15 1.33291e-15
- joint joint_4: limit lower=-3.10862e-14 upper=6.28319 effort=10 velocity=10 -> lower=-3.14159 upper=3.14159 effort=10 velocity=10; origin xyz=-1.11022e-16 -0.076 -0.05 rpy=-1.5708 -6.48265e-16 -1.8837e-16 -> xyz=-1.9521e-17 0.076 -0.05 rpy=1.5708 1.11022e-16 -1.11022e-16
- joint joint_5: limit lower=-0.162156 upper=2.97944 effort=10 velocity=10 -> lower=-1.5708 upper=1.5708 effort=10 velocity=10; origin xyz=-5.55112e-17 1.73472e-18 -0.1125 rpy=-1.5708 -1.84512e-15 -3.11039e-14 -> xyz=-4.31358e-17 -1.73472e-18 -0.1125 rpy=1.5708 -1.5708 0
- joint joint_6: limit lower=-6.28319 upper=0 effort=10 velocity=10 -> lower=-3.14159 upper=3.14159 effort=10 velocity=10; origin xyz=0.0109039 0.0017838 4.27956e-15 rpy=2.97944 1.5708 0 -> xyz=-0.0110489 -8.08314e-19 0 rpy=3.14159 1.5708 0

Commit message: fix frame orientation

File: src/r6bot_description/urdf/robot.urdf (robot description, URDF)
Before this commit: robot robot, 10 links, 9 joints
Joints:
- joint joint_1: origin xyz=7.33525e-17 9.71219e-17 0.1245 rpy=3.14159 -0 1.5708 -> xyz=-9.71219e-17 7.33525e-17 0.1245 rpy=0 -0 3.14159
- joint joint_2: origin xyz=1.2576e-16 0.0895 -0.0575 rpy=1.5708 1.3735e-16 -2.25307e-15 -> xyz=1.17358e-16 -0.0895 0.0575 rpy=1.5708 -1.3735e-16 2.25307e-15
- joint joint_3: origin xyz=4.2689e-08 -0.2 0.0259997 rpy=3.14159 4.65589e-15 1.33291e-15 -> xyz=4.2689e-08 0.2 -0.0259997 rpy=-5.69636e-17 -4.65589e-15 -1.33291e-15
- joint joint_4: origin xyz=-1.9521e-17 0.076 -0.05 rpy=1.5708 1.11022e-16 -1.11022e-16 -> xyz=-1.9521e-17 0.076 -0.05 rpy=-1.5708 1.11022e-16 -1.11022e-16
- joint joint_5: origin xyz=-4.31358e-17 -1.73472e-18 -0.1125 rpy=1.5708 -1.5708 0 -> xyz=-4.66156e-17 3.1225e-17 0.1125 rpy=1.5708 1.5708 0
- joint joint_6: origin xyz=-0.0110489 -8.08314e-19 0 rpy=3.14159 1.5708 0 -> xyz=-0.0110489 4.69647e-18 -1.9082e-17 rpy=-3.24826e-16 -1.5708 0
- joint tool0_tcp_frame: origin xyz=-6.41848e-17 8.44637e-18 0.047085 rpy=-9.35725e-16 -1.99408e-15 -1.96146e-29 -> xyz=-6.41848e-17 8.44637e-18 0.047085 rpy=1.99408e-15 -9.35725e-16 -1.5708
- joint tool1_tcp_frame: origin xyz=-2.15106e-16 2.25417e-16 0.106885 rpy=-2.58091e-15 6.24476e-15 1.5708 -> xyz=-2.15106e-16 2.25417e-16 0.106885 rpy=2.58091e-15 -6.24476e-15 -1.5708
