Commit message: fix naming

File: src/robot_description/urdf/robot.urdf (robot description, URDF)
Before this commit: robot robot, 10 links, 9 joints
Links:
- link link_1: geometry collision mesh filename=package://robot_description/meshes/link_1_collision.stl; visual mesh filename=package://robot_description/meshes/link_1_visual.stl
- link link_2: geometry collision mesh filename=package://robot_description/meshes/link_2_collision.stl; visual mesh filename=package://robot_description/meshes/link_2_visual.stl
- link link_3: geometry collision mesh filename=package://robot_description/meshes/link_3_collision.stl; visual mesh filename=package://robot_description/meshes/link_3_visual.stl
- link link_4: geometry collision mesh filename=package://robot_description/meshes/link_4_collision.stl; visual mesh filename=package://robot_description/meshes/link_4_visual.stl
- link link_5: geometry collision mesh filename=package://robot_description/meshes/link_5_collision.stl; visual mesh filename=package://robot_description/meshes/link_5_visual.stl
- link link_6: geometry collision mesh filename=package://robot_description/meshes/link_6_collision.stl; visual mesh filename=package://robot_description/meshes/link_6_visual.stl
- link link_7: geometry collision mesh filename=package://robot_description/meshes/link_7_collision.stl; visual mesh filename=package://robot_description/meshes/link_7_visual.stl

Commit message: add world frame

File: src/robot_description/urdf/robot.urdf (robot description, URDF)
Before this commit: robot robot, 10 links, 9 joints
Links:
- removed link tool0_tcp
- removed link tool1_tcp
- added link gripper_tcp, mass 1e-9
- added link tool_changer, mass 1e-9
- added link world, mass 1e-9
Joints:
- removed joint tool0_tcp_frame
- removed joint tool1_tcp_frame
- added joint gripper_tcp_frame: type fixed, parent link_7, child gripper_tcp, origin xyz=-2.15106e-16 2.25417e-16 0.106885 rpy=2.58091e-15 -6.24476e-15 -1.5708, axis 0 0 0
- added joint tool_changer_frame: type fixed, parent link_7, child tool_changer, origin xyz=-6.41848e-17 8.44637e-18 0.047085 rpy=1.99408e-15 -9.35725e-16 -1.5708, axis 0 0 0
- added joint world_frame: type fixed, parent link_1, child world, origin xyz=0 -0.35 0 rpy=0 -0 0, axis 0 0 0

Commit message: update 3d model

File: src/robot_description/urdf/robot.urdf (robot description, URDF)
Before this commit: robot robot, 11 links, 10 joints
Links:
- removed link gripper_tcp
- removed link tool_changer
- link link_1: mass 0.552681 -> 0.76382
- link link_2: mass 0.423847 -> 0.633312
- link link_3: mass 0.573947 -> 0.702237
- link link_4: mass 0.28613 -> 0.414775
- link link_5: mass 0.367859 -> 0.382901
- link link_6: mass 0.164337 -> 0.180127
- link link_7: mass 0.117107 -> 0.110548
Joints:
- removed joint gripper_tcp_frame
- removed joint tool_changer_frame
- joint joint_1: origin xyz=-9.71219e-17 7.33525e-17 0.1245 rpy=0 -0 3.14159 -> xyz=-8.56257e-17 6.08362e-17 0.1245 rpy=2.10045e-17 -8.84447e-32 1.5708
- joint joint_2: origin xyz=1.17358e-16 -0.0895 0.0575 rpy=1.5708 -1.3735e-16 2.25307e-15 -> xyz=0.0895 2.21034e-16 0.0575 rpy=1.2285e-14 1.5708 0
- joint joint_3: origin xyz=4.2689e-08 0.2 -0.0259997 rpy=-5.69636e-17 -4.65589e-15 -1.33291e-15 -> xyz=-0.2 4.2689e-08 -0.0259997 rpy=1.06043e-15 -2.77556e-16 1.5708
- joint joint_4: origin xyz=-1.9521e-17 0.076 -0.05 rpy=-1.5708 1.11022e-16 -1.11022e-16 -> xyz=1.26565e-17 0.076 -0.05 rpy=-1.5708 -1.5708 0
- joint joint_5: origin xyz=-4.66156e-17 3.1225e-17 0.1125 rpy=1.5708 1.5708 0 -> xyz=-5.56846e-16 -1.02085e-15 0.1125 rpy=-6.40729e-15 1.5708 0
- joint joint_6: origin xyz=-0.0110489 4.69647e-18 -1.9082e-17 rpy=-3.24826e-16 -1.5708 0 -> xyz=-0.0110489 9.05472e-19 0 rpy=2.7759e-17 -1.5708 0
- joint world_frame: origin xyz=0 -0.35 0 rpy=0 -0 0 -> xyz=-1.42177e-33 -0.35 0 rpy=0 2.10045e-17 5.6569e-32

Commit message: update robot model

File: src/robot_description/urdf/robot.urdf (robot description, URDF)
Before this commit: robot robot, 9 links, 8 joints
Links:
- link link_1: mass 0.76382 -> 0.762917
- link link_2: mass 0.633312 -> 0.632802
- link link_3: mass 0.702237 -> 0.701897
- link link_4: mass 0.414775 -> 0.414434
- link link_5: mass 0.382901 -> 0.382902
- link link_7: mass 0.110548 -> 0.109068
Joints:
- joint joint_1: origin xyz=-8.56257e-17 6.08362e-17 0.1245 rpy=2.10045e-17 -8.84447e-32 1.5708 -> xyz=-9.10289e-17 2.10067e-17 0.1245 rpy=6.85909e-33 -0 1.5708
- joint joint_2: origin xyz=0.0895 2.21034e-16 0.0575 rpy=1.2285e-14 1.5708 0 -> xyz=-0.0895 -1.04373e-16 0.0575 rpy=3.14159 1.5708 0
- joint joint_3: origin xyz=-0.2 4.2689e-08 -0.0259997 rpy=1.06043e-15 -2.77556e-16 1.5708 -> xyz=-0.2 4.2689e-08 -0.0259997 rpy=-7.21645e-15 -1.20516e-14 1.5708
- joint joint_4: origin xyz=1.26565e-17 0.076 -0.05 rpy=-1.5708 -1.5708 0 -> xyz=-3.86347e-16 0.076 -0.05 rpy=-1.5708 -1.5708 0
- joint joint_5: origin xyz=-5.56846e-16 -1.02085e-15 0.1125 rpy=-6.40729e-15 1.5708 0 -> xyz=1.73472e-18 6.57331e-18 0.1125 rpy=9.99201e-16 1.5708 0
- joint joint_6: origin xyz=-0.0110489 9.05472e-19 0 rpy=2.7759e-17 -1.5708 0 -> xyz=-0.0110489 3.75536e-16 -2.55004e-16 rpy=-9.99201e-16 -1.5708 0
- joint world_frame: origin xyz=-1.42177e-33 -0.35 0 rpy=0 2.10045e-17 5.6569e-32 -> xyz=2.17302e-29 -0.35 9.48385e-76 rpy=-2.70967e-75 -8.73725e-47 -6.20864e-29

Commit message: start implementing tool visualization

File: src/robot_description/urdf/robot.urdf (robot description, URDF)
Before this commit: robot robot, 9 links, 8 joints
Links:
- link link_6: mass 0.180127 -> 0.180443
Joints:
- joint joint_1: origin xyz=-9.10289e-17 2.10067e-17 0.1245 rpy=6.85909e-33 -0 1.5708 -> xyz=-0 0 0.1245 rpy=0 0 1.5708
- joint joint_2: origin xyz=-0.0895 -1.04373e-16 0.0575 rpy=3.14159 1.5708 0 -> xyz=-0.0895 -0 0.0575 rpy=-3.14159 1.5708 0
- joint joint_3: origin xyz=-0.2 4.2689e-08 -0.0259997 rpy=-7.21645e-15 -1.20516e-14 1.5708 -> xyz=-0.2 4.2689e-08 -0.0259997 rpy=-0 -0 1.5708
- joint joint_4: limit lower=-3.14159 upper=3.14159 effort=10 velocity=10 -> lower=-2.99773 upper=3.28546 effort=10 velocity=10; origin xyz=-3.86347e-16 0.076 -0.05 rpy=-1.5708 -1.5708 0 -> xyz=-0 0.076 -0.05 rpy=-1.5708 -1.5708 0
- joint joint_5: limit lower=-1.5708 upper=1.5708 effort=10 velocity=10 -> lower=-1.60961 upper=1.53198 effort=10 velocity=10; origin xyz=1.73472e-18 6.57331e-18 0.1125 rpy=9.99201e-16 1.5708 0 -> xyz=0 0 0.1125 rpy=1.5708 1.53198 1.42693
- joint joint_6: limit lower=-3.14159 upper=3.14159 effort=10 velocity=10 -> lower=-1.5382 upper=4.74499 effort=10 velocity=10; origin xyz=-0.0110489 3.75536e-16 -2.55004e-16 rpy=-9.99201e-16 -1.5708 0 -> xyz=-0.0110489 -0 -0 rpy=1.5708 0.0326012 -1.5708
- joint world_frame: origin xyz=2.17302e-29 -0.35 9.48385e-76 rpy=-2.70967e-75 -8.73725e-47 -6.20864e-29 -> xyz=0 -0.35 0 rpy=-0 -0 -0

Commit message: update model

File: src/robot_description/urdf/robot.urdf (robot description, URDF)
Before this commit: robot robot, 9 links, 8 joints
Links:
- removed link link_1
- added link base_plate, mass 0.763578; collision mesh filename=package://robot_description/meshes/base_plate_collision.stl; visual mesh filename=package://robot_description/meshes/base_plate_visual.stl
- link link_2: mass 0.632802 -> 0.6334
- link link_3: mass 0.701897 -> 0.702333
- link link_4: mass 0.414434 -> 0.414871
- link link_5: mass 0.382902 -> 0.387596
- link link_6: mass 0.180127 -> 0.180443
- link link_7: mass 0.109068 -> 0.108782
Joints:
- removed joint base_link_to_link_1
- added joint base_link_to_base_plate: type fixed, parent base_link, child base_plate, origin xyz=0 0 0 rpy=0 -0 0, axis 0 0 1, limit effort=10 velocity=10
- joint joint_1: origin xyz=-9.10289e-17 2.10067e-17 0.1245 rpy=6.85909e-33 -0 1.5708 -> xyz=-0 0.174521 0.1365 rpy=0 -0 0; parent link_1 -> base_plate
- joint joint_2: origin xyz=-0.0895 -1.04373e-16 0.0575 rpy=3.14159 1.5708 0 -> xyz=-0.0895 -0 0.0575 rpy=3.14159 1.5708 0
- joint joint_3: origin xyz=-0.2 4.2689e-08 -0.0259997 rpy=-7.21645e-15 -1.20516e-14 1.5708 -> xyz=-0.2 4.2689e-08 -0.0259997 rpy=-0 -0 1.5708
- joint joint_4: origin xyz=-3.86347e-16 0.076 -0.05 rpy=-1.5708 -1.5708 0 -> xyz=-0 0.076 -0.05 rpy=-1.5708 -1.5708 0
- joint joint_5: origin xyz=1.73472e-18 6.57331e-18 0.1125 rpy=9.99201e-16 1.5708 0 -> xyz=0 -0 0.1125 rpy=0 1.5708 0
- joint joint_6: origin xyz=-0.0110489 3.75536e-16 -2.55004e-16 rpy=-9.99201e-16 -1.5708 0 -> xyz=-0.0110489 0 0 rpy=1.5708 -0 -1.5708
- joint world_frame: origin xyz=2.17302e-29 -0.35 9.48385e-76 rpy=-2.70967e-75 -8.73725e-47 -6.20864e-29 -> xyz=-0.35 0.174521 0.012 rpy=0 -0 -1.5708; parent link_1 -> base_plate

Commit message: update model

File: src/robot_description/urdf/robot.urdf (robot description, URDF)
Before this commit: robot robot, 9 links, 8 joints
Links:
- link base_plate: mass 0.763578 -> 0.824411
- link link_3: mass 0.702333 -> 0.700953
- link link_4: mass 0.414871 -> 0.413336
- link link_5: mass 0.387596 -> 0.404823
- link link_6: mass 0.180443 -> 0.150815
- link link_7: mass 0.108782 -> 0.133959
Joints:
- joint joint_1: origin xyz=-0 0.174521 0.1365 rpy=0 -0 0 -> xyz=-0 0.174521 0.1545 rpy=-0 -0 0
- joint joint_4: origin xyz=-0 0.076 -0.05 rpy=-1.5708 -1.5708 0 -> xyz=0 0.076 -0.05 rpy=-1.5708 -1.5708 0
- joint joint_5: origin xyz=0 -0 0.1125 rpy=0 1.5708 0 -> xyz=0 0 0.124 rpy=0 1.5708 0
- joint joint_6: origin xyz=-0.0110489 0 0 rpy=1.5708 -0 -1.5708 -> xyz=-0.0110489 0 0 rpy=-1.5708 0 1.5708
- joint world_frame: origin xyz=-0.35 0.174521 0.012 rpy=0 -0 -1.5708 -> xyz=-0.35 0.174521 0.012 rpy=-0 -0 -1.5708

Commit message: update model

File: src/robot_description/urdf/robot.urdf (robot description, URDF)
Before this commit: robot robot, 9 links, 8 joints
Joints:
- joint joint_1: origin xyz=-0 0.174521 0.1545 rpy=-0 -0 0 -> xyz=-0 0.174521 0.1545 rpy=0 0 0
- joint joint_5: origin xyz=0 0 0.124 rpy=0 1.5708 0 -> xyz=-0 -0 0.124 rpy=0 1.5708 0
- joint world_frame: origin xyz=-0.35 0.174521 0.012 rpy=-0 -0 -1.5708 -> xyz=-0.35 0.174521 0.012 rpy=0 0 -1.5708
